Commit message: modified tobe_walker, moved transmission macros from gazebo.xacro to tobe.xacro

File: catkin_ws/src/tobe_description/gazebo.xacro (robot description, xacro)
@@ -17,129 +17,3 @@
 		</plugin>
     </gazebo>
-    <xacro:macro name="shoulder_swing_joint_gazebo" params="prefix">
-        <transmission name="${prefix}_shoulder_swing_joint_tran">
-            <type>transmission_interface/SimpleTransmission</type>
-            <joint name="${prefix}_shoulder_swing_joint">
-                <hardwareInterface>hardware_interface/EffortJointInterface</hardwareInterface>
-            </joint>
-            <actuator name="${prefix}_shoulder_swing_joint_motor">
-                <hardwareInterface>hardware_interface/EffortJointInterface</hardwareInterface>
-                <mechanicalReduction>1</mechanicalReduction>
-            </actuator>
-        </transmission>
-    </xacro:macro>
-    <xacro:macro name="shoulder_lateral_joint_gazebo" params="prefix">
-        <transmission name="${prefix}_shoulder_lateral_joint_tran">
-            <type>transmission_interface/SimpleTransmission</type>
-            <joint name="${prefix}_shoulder_lateral_joint">
-                <hardwareInterface>hardware_interface/EffortJointInterface</hardwareInterface>
-            </joint>
-            <actuator name="${prefix}_shoulder_lateral_joint_motor">
-                <hardwareInterface>hardware_interface/EffortJointInterface</hardwareInterface>
-                <mechanicalReduction>1</mechanicalReduction>
-            </actuator>
-        </transmission>
-    </xacro:macro>
-    <xacro:macro name="elbow_joint_gazebo" params="prefix">
-        <transmission name="${prefix}_elbow_joint_tran">
-            <type>transmission_interface/SimpleTransmission</type>
-            <joint name="${prefix}_elbow_joint">
-                <hardwareInterface>hardware_interface/EffortJointInterface</hardwareInterface>
-            </joint>
-            <actuator name="${prefix}_elbow_joint_motor">
-                <hardwareInterface>EffortJointInterface</hardwareInterface>
-                <mechanicalReduction>1</mechanicalReduction>
-            </actuator>
-        </transmission>
-    </xacro:macro>
-    <xacro:macro name="hip_twist_joint_gazebo" params="prefix">
-        <transmission name="${prefix}_hip_twist_joint_tran">
-            <type>transmission_interface/SimpleTransmission</type>
-            <joint name="${prefix}_hip_twist_joint">
-                <hardwareInterface>hardware_interface/EffortJointInterface</hardwareInterface>
-            </joint>
-            <actuator name="${prefix}_hip_twist_joint_motor">
-                <hardwareInterface>hardware_interface/EffortJointInterface</hardwareInterface>
-                <mechanicalReduction>1</mechanicalReduction>
-            </actuator>
-        </transmission>
-    </xacro:macro>
-    <xacro:macro name="hip_lateral_joint_gazebo" params="prefix">
-        <transmission name="${prefix}_hip_lateral_joint_tran">
-            <type>transmission_interface/SimpleTransmission</type>
-            <joint name="${prefix}_hip_lateral_joint">
-                <hardwareInterface>hardware_interface/EffortJointInterface</hardwareInterface>
-            </joint>
-            <actuator name="${prefix}_hip_lateral_joint_motor">
-                <hardwareInterface>hardware_interface/EffortJointInterface</hardwareInterface>
-                <mechanicalReduction>1</mechanicalReduction>
-            </actuator>
-        </transmission>
-    </xacro:macro>
-    <xacro:macro name="hip_swing_joint_gazebo" params="prefix">
-        <transmission name="${prefix}_hip_swing_joint_tran">
-            <type>transmission_interface/SimpleTransmission</type>
-            <joint name="${prefix}_hip_swing_joint">
-                <hardwareInterface>hardware_interface/EffortJointInterface</hardwareInterface>
-            </joint>
-            <actuator name="${prefix}_hip_swing_joint_motor">
-                <hardwareInterface>hardware_interface/EffortJointInterface</hardwareInterface>
-                <mechanicalReduction>1</mechanicalReduction>
-            </actuator>
-        </transmission>
-    </xacro:macro>
-    <xacro:macro name="knee_joint_gazebo" params="prefix">
-        <transmission name="${prefix}_knee_joint_tran">
-            <type>transmission_interface/SimpleTransmission</type>
-            <joint name="${prefix}_knee_joint">
-                <hardwareInterface>hardware_interface/EffortJointInterface</hardwareInterface>
-            </joint>
-            <actuator name="${prefix}_knee_joint_motor">
-                <hardwareInterface>hardware_interface/EffortJointInterface</hardwareInterface>
-                <mechanicalReduction>1</mechanicalReduction>
-            </actuator>
-        </transmission>
-    </xacro:macro>
-    <xacro:macro name="ankle_swing_joint_gazebo" params="prefix">
-        <transmission name="${prefix}_ankle_swing_joint_tran">
-            <type>transmission_interface/SimpleTransmission</type>
-            <joint name="${prefix}_ankle_swing_joint">
-                <hardwareInterface>hardware_interface/EffortJointInterface</hardwareInterface>
-            </joint>
-            <actuator name="${prefix}_ankle_swing_joint_motor">
-                <hardwareInterface>hardware_interface/EffortJointInterface</hardwareInterface>
-                <mechanicalReduction>1</mechanicalReduction>
-            </actuator>
-        </transmission>
-    </xacro:macro>
-    <xacro:macro name="ankle_lateral_joint_gazebo" params="prefix">
-        <transmission name="${prefix}_ankle_lateral_joint_tran">
-            <type>transmission_interface/SimpleTransmission</type>
-            <joint name="${prefix}_ankle_lateral_joint">
-                <hardwareInterface>hardware_interface/EffortJointInterface</hardwareInterface>
-            </joint>
-            <actuator name="${prefix}_ankle_lateral_joint_motor">
-                <hardwareInterface>hardware_interface/EffortJointInterface</hardwareInterface>
-                <mechanicalReduction>1</mechanicalReduction>
-            </actuator>
-        </transmission>
-    </xacro:macro>
-    <xacro:shoulder_swing_joint_gazebo prefix="r"/>
-    <xacro:shoulder_swing_joint_gazebo prefix="l"/>
-    <xacro:shoulder_lateral_joint_gazebo prefix="r"/>
-    <xacro:shoulder_lateral_joint_gazebo prefix="l"/>
-    <xacro:elbow_joint_gazebo prefix="r"/>
-    <xacro:elbow_joint_gazebo prefix="l"/>
-    <xacro:hip_twist_joint_gazebo prefix="r"/>
-    <xacro:hip_twist_joint_gazebo prefix="l"/>
-    <xacro:hip_lateral_joint_gazebo prefix="r"/>
-    <xacro:hip_lateral_joint_gazebo prefix="l"/>
-    <xacro:hip_swing_joint_gazebo prefix="r"/>
-    <xacro:hip_swing_joint_gazebo prefix="l"/>
-    <xacro:knee_joint_gazebo prefix="r"/>
-    <xacro:knee_joint_gazebo prefix="l"/>
-    <xacro:ankle_swing_joint_gazebo prefix="r"/>
-    <xacro:ankle_swing_joint_gazebo prefix="l"/>
-    <xacro:ankle_lateral_joint_gazebo prefix="r"/>
-    <xacro:ankle_lateral_joint_gazebo prefix="l"/>
 </robot>

File: catkin_ws/src/tobe_description/tobe.xacro (robot description, xacro)
@@ -628,3 +628,129 @@
     <!-- Left ankle lateral to foot -->
     <xacro:foot_joint prefix="l" reflect="-1"/>
+    <xacro:macro name="shoulder_swing_joint_gazebo" params="prefix">
+        <transmission name="${prefix}_shoulder_swing_joint_tran">
+            <type>transmission_interface/SimpleTransmission</type>
+            <joint name="${prefix}_shoulder_swing_joint">
+                <hardwareInterface>hardware_interface/EffortJointInterface</hardwareInterface>
+            </joint>
+            <actuator name="${prefix}_shoulder_swing_joint_motor">
+                <hardwareInterface>hardware_interface/EffortJointInterface</hardwareInterface>
+                <mechanicalReduction>1</mechanicalReduction>
+            </actuator>
+        </transmission>
+    </xacro:macro>
+    <xacro:macro name="shoulder_lateral_joint_gazebo" params="prefix">
+        <transmission name="${prefix}_shoulder_lateral_joint_tran">
+            <type>transmission_interface/SimpleTransmission</type>
+            <joint name="${prefix}_shoulder_lateral_joint">
+                <hardwareInterface>hardware_interface/EffortJointInterface</hardwareInterface>
+            </joint>
+            <actuator name="${prefix}_shoulder_lateral_joint_motor">
+                <hardwareInterface>hardware_interface/EffortJointInterface</hardwareInterface>
+                <mechanicalReduction>1</mechanicalReduction>
+            </actuator>
+        </transmission>
+    </xacro:macro>
+    <xacro:macro name="elbow_joint_gazebo" params="prefix">
+        <transmission name="${prefix}_elbow_joint_tran">
+            <type>transmission_interface/SimpleTransmission</type>
+            <joint name="${prefix}_elbow_joint">
+                <hardwareInterface>hardware_interface/EffortJointInterface</hardwareInterface>
+            </joint>
+            <actuator name="${prefix}_elbow_joint_motor">
+                <hardwareInterface>EffortJointInterface</hardwareInterface>
+                <mechanicalReduction>1</mechanicalReduction>
+            </actuator>
+        </transmission>
+    </xacro:macro>
+    <xacro:macro name="hip_twist_joint_gazebo" params="prefix">
+        <transmission name="${prefix}_hip_twist_joint_tran">
+            <type>transmission_interface/SimpleTransmission</type>
+            <joint name="${prefix}_hip_twist_joint">
+                <hardwareInterface>hardware_interface/EffortJointInterface</hardwareInterface>
+            </joint>
+            <actuator name="${prefix}_hip_twist_joint_motor">
+                <hardwareInterface>hardware_interface/EffortJointInterface</hardwareInterface>
+                <mechanicalReduction>1</mechanicalReduction>
+            </actuator>
+        </transmission>
+    </xacro:macro>
+    <xacro:macro name="hip_lateral_joint_gazebo" params="prefix">
+        <transmission name="${prefix}_hip_lateral_joint_tran">
+            <type>transmission_interface/SimpleTransmission</type>
+            <joint name="${prefix}_hip_lateral_joint">
+                <hardwareInterface>hardware_interface/EffortJointInterface</hardwareInterface>
+            </joint>
+            <actuator name="${prefix}_hip_lateral_joint_motor">
+                <hardwareInterface>hardware_interface/EffortJointInterface</hardwareInterface>
+                <mechanicalReduction>1</mechanicalReduction>
+            </actuator>
+        </transmission>
+    </xacro:macro>
+    <xacro:macro name="hip_swing_joint_gazebo" params="prefix">
+        <transmission name="${prefix}_hip_swing_joint_tran">
+            <type>transmission_interface/SimpleTransmission</type>
+            <joint name="${prefix}_hip_swing_joint">
+                <hardwareInterface>hardware_interface/EffortJointInterface</hardwareInterface>
+            </joint>
+            <actuator name="${prefix}_hip_swing_joint_motor">
+                <hardwareInterface>hardware_interface/EffortJointInterface</hardwareInterface>
+                <mechanicalReduction>1</mechanicalReduction>
+            </actuator>
+        </transmission>
+    </xacro:macro>
+    <xacro:macro name="knee_joint_gazebo" params="prefix">
+        <transmission name="${prefix}_knee_joint_tran">
+            <type>transmission_interface/SimpleTransmission</type>
+            <joint name="${prefix}_knee_joint">
+                <hardwareInterface>hardware_interface/EffortJointInterface</hardwareInterface>
+            </joint>
+            <actuator name="${prefix}_knee_joint_motor">
+                <hardwareInterface>hardware_interface/EffortJointInterface</hardwareInterface>
+                <mechanicalReduction>1</mechanicalReduction>
+            </actuator>
+        </transmission>
+    </xacro:macro>
+    <xacro:macro name="ankle_swing_joint_gazebo" params="prefix">
+        <transmission name="${prefix}_ankle_swing_joint_tran">
+            <type>transmission_interface/SimpleTransmission</type>
+            <joint name="${prefix}_ankle_swing_joint">
+                <hardwareInterface>hardware_interface/EffortJointInterface</hardwareInterface>
+            </joint>
+            <actuator name="${prefix}_ankle_swing_joint_motor">
+                <hardwareInterface>hardware_interface/EffortJointInterface</hardwareInterface>
+                <mechanicalReduction>1</mechanicalReduction>
+            </actuator>
+        </transmission>
+    </xacro:macro>
+    <xacro:macro name="ankle_lateral_joint_gazebo" params="prefix">
+        <transmission name="${prefix}_ankle_lateral_joint_tran">
+            <type>transmission_interface/SimpleTransmission</type>
+            <joint name="${prefix}_ankle_lateral_joint">
+                <hardwareInterface>hardware_interface/EffortJointInterface</hardwareInterface>
+            </joint>
+            <actuator name="${prefix}_ankle_lateral_joint_motor">
+                <hardwareInterface>hardware_interface/EffortJointInterface</hardwareInterface>
+                <mechanicalReduction>1</mechanicalReduction>
+            </actuator>
+        </transmission>
+    </xacro:macro>
+    <xacro:shoulder_swing_joint_gazebo prefix="r"/>
+    <xacro:shoulder_swing_joint_gazebo prefix="l"/>
+    <xacro:shoulder_lateral_joint_gazebo prefix="r"/>
+    <xacro:shoulder_lateral_joint_gazebo prefix="l"/>
+    <xacro:elbow_joint_gazebo prefix="r"/>
+    <xacro:elbow_joint_gazebo prefix="l"/>
+    <xacro:hip_twist_joint_gazebo prefix="r"/>
+    <xacro:hip_twist_joint_gazebo prefix="l"/>
+    <xacro:hip_lateral_joint_gazebo prefix="r"/>
+    <xacro:hip_lateral_joint_gazebo prefix="l"/>
+    <xacro:hip_swing_joint_gazebo prefix="r"/>
+    <xacro:hip_swing_joint_gazebo prefix="l"/>
+    <xacro:knee_joint_gazebo prefix="r"/>
+    <xacro:knee_joint_gazebo prefix="l"/>
+    <xacro:ankle_swing_joint_gazebo prefix="r"/>
+    <xacro:ankle_swing_joint_gazebo prefix="l"/>
+    <xacro:ankle_lateral_joint_gazebo prefix="r"/>
+    <xacro:ankle_lateral_joint_gazebo prefix="l"/>
 </robot>
